Commit message: replace orginal franka grippers with finray

File: franka_description/robots/hand_original.xacro (robot description, xacro)
@@ -25,7 +25,6 @@
     <link name="${arm_id}_leftfinger">
       <visual>
-      <origin xyz="0. 0. 0" rpy="0 0 ${pi}"/>
         <geometry>
-          <mesh filename="package://${description_pkg}/meshes/visual/one_piece_thin_grasp_finray_finger.obj" />
+          <mesh filename="package://${description_pkg}/meshes/visual/finger.dae" />
         </geometry>
       </visual>
@@ -64,7 +63,7 @@
     <link name="${arm_id}_rightfinger">
       <visual>
-        <origin xyz="0.0 -0.0 0" rpy="0 0 0" />
+        <origin xyz="0 0 0" rpy="0 0 ${pi}" />
         <geometry>
-          <mesh filename="package://${description_pkg}/meshes/visual/one_piece_thin_grasp_finray_finger.obj" />
+          <mesh filename="package://${description_pkg}/meshes/visual/finger.dae" />
         </geometry>
       </visual>
